Commit message: Use urdf-loader library for proper URDF parsing
- Install urdf-loader package that handles URDF transforms correctly
- Move STL files to assets/ subfolder to match URDF paths
- Remove waveshare mounting plate (STL not available)
- Loader handles all coordinate transforms automatically
- Joint positions updated via setJointValue()

🤖 Generated with [Claude Code](https://claude.com/claude-code)

Co-Authored-By: Claude <noreply@anthropic.com>

File: public/models/so101/so101.urdf (robot description, URDF)
Before this commit: robot so101_new_calib, 8 links, 7 joints
Links:
- link base_link: geometry collision mesh filename=assets/base_motor_holder_so101_v1.stl; collision mesh filename=assets/base_so101_v2.stl
